File: Power Subsystem/Power Subsystem.kicad_pcb (KiCad board)
At the start: 2 copper layers, 32.5 x 32.5 mm, 0 parts

Commit message: Final Schematic and PCB designs
Parts:
- added +5V1: TestPoint, TestPoint:TestPoint_Keystone_5019_Minature, F.Cu at (141.4, 64.4)
- added +BATT1: TestPoint, TestPoint:TestPoint_Keystone_5019_Minature, F.Cu at (149.6, 73.7)
- added C1: 4.7µF, Capacitor_SMD:C_0402_1005Metric, F.Cu at (149.4, 54.8)
- added C2: 4.7µF, Capacitor_SMD:C_0402_1005Metric, F.Cu at (149.4, 55.9)
- added C3: 100nF, Capacitor_SMD:C_0402_1005Metric, F.Cu at (141.7, 52.3)
- added C4: 100nF, Capacitor_SMD:C_0402_1005Metric, F.Cu at (157.3, 52.3)
- added D1: LED, LED_SMD:LED_0603_1608Metric, F.Cu at (146.4, 50.1)
- added GND1: TestPoint, TestPoint:TestPoint_Keystone_5019_Minature, F.Cu at (142.2, 73.7)
- added J1: Conn_01x16_Pin, Connector_PinHeader_2.54mm:PinHeader_2x08_P2.54mm_Vertical, B.Cu at (158.5, 45.2)
- added J2: Conn_01x02_Pin, Connector_JST:JST_PH_S2B-PH-K_1x02_P2.00mm_Horizontal, F.Cu at (165.1, 65.3)
- added JP1: Jumper_2_Bridged, Jumper:SolderJumper-2_P1.3mm_Bridged2Bar_RoundedPad1.0x1.5mm, F.Cu at (165.7, 68.8)
- added JP11: Jumper_2_Open, Jumper:SolderJumper-2_P1.3mm_Open_TrianglePad1.0x1.5mm, F.Cu at (144.9, 67.8)
- added JP13: Jumper_2_Bridged, Jumper:SolderJumper-2_P1.3mm_Bridged2Bar_RoundedPad1.0x1.5mm, F.Cu at (146.9, 55.3)
- added JP2: Jumper_2_Open, Jumper:SolderJumper-2_P1.3mm_Open_TrianglePad1.0x1.5mm, F.Cu at (151.5, 59.4)
- added JP5: Jumper_2_Open, Jumper:SolderJumper-2_P1.3mm_Open_TrianglePad1.0x1.5mm, F.Cu at (151.5, 63.5)
- added JP8: Jumper_2_Open, Jumper:SolderJumper-2_P1.3mm_Open_TrianglePad1.0x1.5mm, F.Cu at (151.4, 67.8)
- added Motor2_B1: TestPoint, TestPoint:TestPoint_Keystone_5019_Minature, F.Cu at (135.4, 73.4)
- added Motor_1: DRV8837, Package_SON:WSON-8-1EP_2x2mm_P0.5mm_EP0.9x1.6mm, F.Cu at (141.7, 50.5)
- added Motor_1A1: TestPoint, TestPoint:TestPoint_Keystone_5019_Minature, F.Cu at (135.4, 61.6)
- added Motor_1B1: TestPoint, TestPoint:TestPoint_Keystone_5019_Minature, F.Cu at (135.4, 64.5)
- added Motor_2: DRV8837, Package_SON:WSON-8-1EP_2x2mm_P0.5mm_EP0.9x1.6mm, F.Cu at (157.2, 50.5)
- added Motor_2A1: TestPoint, TestPoint:TestPoint_Keystone_5019_Minature, F.Cu at (135.4, 70.2)
- added PWM1: TestPoint, TestPoint:TestPoint_Keystone_5019_Minature, F.Cu at (157.5, 57.0)
- added PWM2: TestPoint, TestPoint:TestPoint_Keystone_5019_Minature, F.Cu at (157.5, 60.0)
- added PWM3: TestPoint, TestPoint:TestPoint_Keystone_5019_Minature, F.Cu at (141.7, 57.0)
- added PWM4: TestPoint, TestPoint:TestPoint_Keystone_5019_Minature, F.Cu at (141.7, 59.9)
- added R10: 3k, Resistor_SMD:R_0603_1608Metric, F.Cu at (148.2, 66.9)
- added R11: 3k, Resistor_SMD:R_0603_1608Metric, F.Cu at (148.2, 68.3)
- added R2: 6.8k, Resistor_SMD:R_0603_1608Metric, F.Cu at (148.0, 58.9)
- added R3: 6.8k, Resistor_SMD:R_0603_1608Metric, F.Cu at (148.0, 60.6)
- added R4: 470, Resistor_SMD:R_0402_1005Metric, F.Cu at (147.9, 62.7)
- added R5: 470, Resistor_SMD:R_0402_1005Metric, F.Cu at (147.9, 64.0)
- added R7: 1.2k, Resistor_SMD:R_0603_1608Metric, F.Cu at (154.6, 66.9)
- added R8: 1.2k, Resistor_SMD:R_0603_1608Metric, F.Cu at (154.6, 68.3)
- added SW1: SW_SPDT_312, Custom Footprints:SW-TH_SS-12D10L5, F.Cu at (161.0, 73.9)
- added U1: MCP73831-2-OT, Package_TO_SOT_SMD:SOT-23-5, F.Cu at (149.5, 51.1)
Routing:
- net +BATT: track 0.00 -> 98.4 mm, vias 0 -> 6
- net Motor2_A: track 0.00 -> 47.1 mm, vias 0 -> 2
- net Motor2_B: track 0.00 -> 46.7 mm, vias 0 -> 2
- net +5V: track 0.00 -> 40.9 mm, vias 0 -> 4
- net Motor1_B: track 0.00 -> 35.0 mm, vias 0 -> 1
- net BATT_ADC: track 0.00 -> 32.3 mm, vias 0 -> 1
- net Motor1_A: track 0.00 -> 28.4 mm, vias 0 -> 1
- net PWM2: track 0.00 -> 26.7 mm
- net PWM4: track 0.00 -> 25.3 mm
- net PWM1: track 0.00 -> 19.4 mm, vias 0 -> 2
- net PWM3: track 0.00 -> 18.0 mm, vias 0 -> 2
- net Net-(U1-PROG): track 0.00 -> 15.7 mm, vias 0 -> 2
- net Net-(JP13-A): track 0.00 -> 13.1 mm
- net Net-(J2-Pin_1): track 0.00 -> 12.3 mm
- net Net-(D1-A): track 0.00 -> 6.02 mm, vias 0 -> 2
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- added copper zone on B.Cu, net GND
- added copper zone on F.Cu, net GND
Other:
- board size 32.5 x 32.5 mm -> 36.3 x 37.2 mm
